File: hardware/minimax.kicad_pcb (KiCad board)
At the start: 4 copper layers, 35 x 40 mm, 60 parts, among them J1 524352271, J2 59S1AC-40MT5-Z, J3 PRT-14417, J4 PRT-14417, Q1 DMG1012T, Q2 DMG1012T, Q3 DMG1012T, U1 MAX96717GTJ/VY+, U2 MAX20049ATED/VY+

Commit message: submitted for board fab
Parts:
- R18: value 5.1K -> 402
- R6: value 402 -> 5.1K
- moved R4 13.5 mm to (157.6, 105.7), turned to 180 degrees
- moved R17 13.5 mm to (145.2, 100.3), turned to 0 degrees
- moved R6 10.6 mm to (157.6, 104.5)
- moved R18 10.5 mm to (147.4, 107.3), turned to 180 degrees
- moved C5 0.05 mm to (153.7, 108.1)
- moved C6 0.05 mm to (154.8, 108.1)
- moved C7 0.05 mm to (157.0, 108.1)
- renumbered MFP3 to MFP6, MFP2 to MFP7, MFP1 to MFP8
Connections:
- Q1 pad 1: /gmsl/ERRB -> /gmsl/LOCK
- Q2 pad 1: /gmsl/LOCK -> /gmsl/ERRB
- R17 pad 2: /gmsl/LOCK -> Net-(U1-PWDNB)
- R18 pad 1: VDDIO -> Net-(U1-XRES)
- R18 pad 2: /gmsl/ERRB -> GND
- R4 pad 2: Net-(U1-PWDNB) -> /gmsl/LOCK
- R6 pad 1: Net-(U1-XRES) -> VDDIO
- R6 pad 2: GND -> /gmsl/ERRB
Routing:
- net VDDIO: track 66.5 -> 59.3 mm
- net /gmsl/ERRB: track 30.3 -> 35.2 mm, vias 3 -> 2
- net /camera/POWER_EN: track 21.4 -> 17.2 mm
- net /gmsl/LOCK: track 34.0 -> 32.3 mm, vias 3 -> 2
- net /camera/LED_EN: track 18.1 -> 19.0 mm
- net GND: track 18.8 -> 19.3 mm, vias 33 -> 56
- added copper zone on In2.Cu, net +1V2
- added copper zone on In2.Cu, net +1V8
- added copper zone on In2.Cu, net VDDIO
